Commit message: testing models

File: abb_irb6640_support/urdf/irb6640_185_280.urdf (robot description, URDF)
Before this commit: robot abb_irb6640_185_280, 11 links, 10 joints
Links:
- link base_link: geometry collision mesh filename=package://abb_irb6640_support/meshes/irb6640/collision/base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; visual mesh filename=package://abb_irb6640_support/meshes/irb6640/visual/base_li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
- link link_1: geometry collision mesh filename=package://abb_irb6640_support/meshes/irb6640/collision/link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; visual mesh filename=package://abb_irb6640_support/meshes/irb6640/visual/link_1.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
- link link_2: geometry collision mesh filename=package://abb_irb6640_support/meshes/irb6640/collision/link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; visual mesh filename=package://abb_irb6640_support/meshes/irb6640/visual/link_2.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
- link link_3: geometry collision mesh filename=package://abb_irb6640_support/meshes/irb6640/collision/link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; visual mesh filename=package://abb_irb6640_support/meshes/irb6640/visual/link_3.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
- link link_5: geometry collision mesh filename=package://abb_irb6640_support/meshes/irb6640/collision/link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; visual mesh filename=package://abb_irb6640_support/meshes/irb6640/visual/link_5.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
- link link_6: geometry collision mesh filename=package://abb_irb6640_support/meshes/irb6640/collision/link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; visual mesh filename=package://abb_irb6640_support/meshes/irb6640/visual/link_6.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
- link link_cylinder: geometry collision mesh filename=package://abb_irb6640_support/meshes/irb6640/collision/cyli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; visual mesh filename=package://abb_irb6640_support/meshes/irb6640/visual/cylinde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
- link link_piston: geometry collision mesh filename=package://abb_irb6640_support/meshes/irb6640/collision/pist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; visual mesh filename=package://abb_irb6640_support/meshes/irb6640/visual/piston_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

File: abb_irb6640_support/urdf/irb6640_185_280_macro.xacro (robot description, xacro)
@@ -6,10 +6,10 @@
       <collision name="collision">
         <geometry>
-          <mesh filename="package://abb_irb6640_support/meshes/irb6640_185_280/collision/base_link.stl"/>
+          <mesh filename="package://abb_irb6640_support/meshes/irb6640/collision/base_link.stl"/>
         </geometry>
       </collision>
       <visual name="visual">
         <geometry>
-          <mesh filename="package://abb_irb6640_support/meshes/irb6640_185_280/visual/base_link.dae"/>
+          <mesh filename="package://abb_irb6640_support/meshes/irb6640/visual/base_link.dae"/>
         </geometry>
         <material name="yellow">
@@ -21,10 +21,10 @@
       <collision name="collision">
         <geometry>
-          <mesh filename="package://abb_irb6640_support/meshes/irb6640_185_280/collision/link_1.stl"/>
+          <mesh filename="package://abb_irb6640_support/meshes/irb6640/collision/link_1.stl"/>
         </geometry>
       </collision>
       <visual name="visual">
         <geometry>
-          <mesh filename="package://abb_irb6640_support/meshes/irb6640_185_280/visual/link_1.dae"/>
+          <mesh filename="package://abb_irb6640_support/meshes/irb6640/visual/link_1.dae"/>
         </geometry>
         <material name="yellow"/>
@@ -34,10 +34,10 @@
       <collision name="collision">
         <geometry>
-          <mesh filename="package://abb_irb6640_support/meshes/irb6640_185_280/collision/link_2.stl"/>
+          <mesh filename="package://abb_irb6640_support/meshes/irb6640/collision/link_2.stl"/>
         </geometry>
       </collision>
       <visual name="visual">
         <geometry>
-          <mesh filename="package://abb_irb6640_support/meshes/irb6640_185_280/visual/link_2.dae"/>
+          <mesh filename="package://abb_irb6640_support/meshes/irb6640/visual/link_2.dae"/>
         </geometry>
         <material name="yellow"/>
@@ -47,10 +47,10 @@
       <collision name="collision">
         <geometry>
-          <mesh filename="package://abb_irb6640_support/meshes/irb6640_185_280/collision/link_3.stl"/>
+          <mesh filename="package://abb_irb6640_support/meshes/irb6640/collision/link_3.stl"/>
         </geometry>
       </collision>
       <visual name="visual">
         <geometry>
-          <mesh filename="package://abb_irb6640_support/meshes/irb6640_185_280/visual/link_3.dae"/>
+          <mesh filename="package://abb_irb6640_support/meshes/irb6640/visual/link_3.dae"/>
         </geometry>
         <material name="yellow"/>
@@ -73,10 +73,10 @@
       <collision name="collision">
         <geometry>
-          <mesh filename="package://abb_irb6640_support/meshes/irb6640_185_280/collision/link_5.stl"/>
+          <mesh filename="package://abb_irb6640_support/meshes/irb6640/collision/link_5.stl"/>
         </geometry>
       </collision>
       <visual name="visual">
         <geometry>
-          <mesh filename="package://abb_irb6640_support/meshes/irb6640_185_280/visual/link_5.dae"/>
+          <mesh filename="package://abb_irb6640_support/meshes/irb6640/visual/link_5.dae"/>
         </geometry>
         <material name="yellow"/>
@@ -86,10 +86,10 @@
       <collision name="collision">
         <geometry>
-          <mesh filename="package://abb_irb6640_support/meshes/irb6640_185_280/collision/link_6.stl"/>
+          <mesh filename="package://abb_irb6640_support/meshes/irb6640/collision/link_6.stl"/>
         </geometry>
       </collision>
       <visual name="visual">
         <geometry>
-          <mesh filename="package://abb_irb6640_support/meshes/irb6640_185_280/visual/link_6.dae"/>
+          <mesh filename="package://abb_irb6640_support/meshes/irb6640/visual/link_6.dae"/>
         </geometry>
         <material name="yellow"/>
@@ -101,10 +101,10 @@
       <collision name="collision">
         <geometry>
-          <mesh filename="package://abb_irb6640_support/meshes/irb6640_185_280/collision/cylinder_link.stl"/>
+          <mesh filename="package://abb_irb6640_support/meshes/irb6640/collision/cylinder_link.stl"/>
         </geometry>
       </collision>
       <visual name="visual">
         <geometry>
-          <mesh filename="package://abb_irb6640_support/meshes/irb6640_185_280/visual/cylinder_link.dae"/>
+          <mesh filename="package://abb_irb6640_support/meshes/irb6640/visual/cylinder_link.dae"/>
         </geometry>
         <material name="yellow"/>
@@ -114,10 +114,10 @@
       <collision name="collision">
         <geometry>
-          <mesh filename="package://abb_irb6640_support/meshes/irb6640_185_280/collision/piston_link.stl"/>
+          <mesh filename="package://abb_irb6640_support/meshes/irb6640/collision/piston_link.stl"/>
         </geometry>
       </collision>
       <visual name="visual">
         <geometry>
-          <mesh filename="package://abb_irb6640_support/meshes/irb6640_185_280/visual/piston_link.dae"/>
+          <mesh filename="package://abb_irb6640_support/meshes/irb6640/visual/piston_link.dae"/>
         </geometry>
         <material name="yellow"/>

File: abb_irb6640_support/urdf/irb6640_235_255_macro.xacro (robot description, xacro)
@@ -6,10 +6,10 @@
       <collision name="collision">
         <geometry>
-          <mesh filename="package://abb_irb6640_support/meshes/irb6640_235_255/collision/base_link.stl"/>
+          <mesh filename="package://abb_irb6640_support/meshes/irb6640/collision/base_link.stl"/>
         </geometry>
       </collision>
       <visual name="visual">
         <geometry>
-          <mesh filename="package://abb_irb6640_support/meshes/irb6640_235_255/visual/base_link.dae"/>
+          <mesh filename="package://abb_irb6640_support/meshes/irb6640/visual/base_link.dae"/>
         </geometry>
         <material name="yellow">
@@ -21,10 +21,10 @@
       <collision name="collision">
         <geometry>
-          <mesh filename="package://abb_irb6640_support/meshes/irb6640_235_255/collision/link_1.stl"/>
+          <mesh filename="package://abb_irb6640_support/meshes/irb6640/collision/link_1.stl"/>
         </geometry>
       </collision>
       <visual name="visual">
         <geometry>
-          <mesh filename="package://abb_irb6640_support/meshes/irb6640_235_255/visual/link_1.dae"/>
+          <mesh filename="package://abb_irb6640_support/meshes/irb6640/visual/link_1.dae"/>
         </geometry>
         <material name="yellow"/>
@@ -34,10 +34,10 @@
       <collision name="collision">
         <geometry>
-          <mesh filename="package://abb_irb6640_support/meshes/irb6640_235_255/collision/link_2.stl"/>
+          <mesh filename="package://abb_irb6640_support/meshes/irb6640/collision/link_2.stl"/>
         </geometry>
       </collision>
       <visual name="visual">
         <geometry>
-          <mesh filename="package://abb_irb6640_support/meshes/irb6640_235_255/visual/link_2.dae"/>
+          <mesh filename="package://abb_irb6640_support/meshes/irb6640/visual/link_2.dae"/>
         </geometry>
         <material name="yellow"/>
@@ -47,10 +47,10 @@
       <collision name="collision">
         <geometry>
-          <mesh filename="package://abb_irb6640_support/meshes/irb6640_235_255/collision/link_3.stl"/>
+          <mesh filename="package://abb_irb6640_support/meshes/irb6640/collision/link_3.stl"/>
         </geometry>
       </collision>
       <visual name="visual">
         <geometry>
-          <mesh filename="package://abb_irb6640_support/meshes/irb6640_235_255/visual/link_3.dae"/>
+          <mesh filename="package://abb_irb6640_support/meshes/irb6640/visual/link_3.dae"/>
         </geometry>
         <material name="yellow"/>
@@ -73,10 +73,10 @@
       <collision name="collision">
         <geometry>
-          <mesh filename="package://abb_irb6640_support/meshes/irb6640_235_255/collision/link_5.stl"/>
+          <mesh filename="package://abb_irb6640_support/meshes/irb6640/collision/link_5.stl"/>
         </geometry>
       </collision>
       <visual name="visual">
         <geometry>
-          <mesh filename="package://abb_irb6640_support/meshes/irb6640_235_255/visual/link_5.dae"/>
+          <mesh filename="package://abb_irb6640_support/meshes/irb6640/visual/link_5.dae"/>
         </geometry>
         <material name="yellow"/>
@@ -86,10 +86,10 @@
       <collision name="collision">
         <geometry>
-          <mesh filename="package://abb_irb6640_support/meshes/irb6640_235_255/collision/link_6.stl"/>
+          <mesh filename="package://abb_irb6640_support/meshes/irb6640/collision/link_6.stl"/>
         </geometry>
       </collision>
       <visual name="visual">
         <geometry>
-          <mesh filename="package://abb_irb6640_support/meshes/irb6640_235_255/visual/link_6.dae"/>
+          <mesh filename="package://abb_irb6640_support/meshes/irb6640/visual/link_6.dae"/>
         </geometry>
         <material name="yellow"/>
@@ -101,10 +101,10 @@
       <collision name="collision">
         <geometry>
-          <mesh filename="package://abb_irb6640_support/meshes/irb6640_235_255/collision/cylinder_link.stl"/>
+          <mesh filename="package://abb_irb6640_support/meshes/irb6640/collision/cylinder_link.stl"/>
         </geometry>
       </collision>
       <visual name="visual">
         <geometry>
-          <mesh filename="package://abb_irb6640_support/meshes/irb6640_235_255/visual/cylinder_link.dae"/>
+          <mesh filename="package://abb_irb6640_support/meshes/irb6640/visual/cylinder_link.dae"/>
         </geometry>
         <material name="yellow"/>
@@ -114,10 +114,10 @@
       <collision name="collision">
         <geometry>
-          <mesh filename="package://abb_irb6640_support/meshes/irb6640_235_255/collision/piston_link.stl"/>
+          <mesh filename="package://abb_irb6640_support/meshes/irb6640/collision/piston_link.stl"/>
         </geometry>
       </collision>
       <visual name="visual">
         <geometry>
-          <mesh filename="package://abb_irb6640_support/meshes/irb6640_235_255/visual/piston_link.dae"/>
+          <mesh filename="package://abb_irb6640_support/meshes/irb6640/visual/piston_link.dae"/>
         </geometry>
         <material name="yellow"/>
